File: Schematic/STM32F405 Flight Controller.kicad_sch (KiCad schematic)
At the start: 72 parts, among them J1 USB_C_Receptacle_USB2.0_16P, J2 XT60 (BATT), J3 ESC_1, J4 ESC_2, J5 ESC_3, J6 ESC_4, J7 SWD, SW1 SW_Push, SW2 SW_Push, U1 STM32F405RGTx, U2 MPU-6050, U3 BMP280, U4 AP7361C-33E, U5 LIS3MDL, U7 LMR33640DDDA, U8 W25Q128JVS, Y1 16MHz Crystal

Commit message: Add files via upload
Updated schematic
Parts:
- added R12: 10k, Resistor_SMD:R_0603_1608Metric, symbol Device:R
- C10, C11, C26, C27, C8, C9: footprint Capacitor_SMD:C_0805_2012Metric -> Capacitor_SMD:C_0603_1608Metric
- C15, C16: footprint PCM_Capacitor_SMD_AKL:C_0402_1005Metric -> Capacitor_SMD:C_0603_1608Metric
- C17: footprint Capacitor_SMD:C_0402_1005Metric -> Capacitor_SMD:C_0603_1608Metric
- D3: footprint LED_THT:LED_D3.0mm_FlatTop -> LED_SMD:LED_0805_2012Metric
- SW1, SW2: footprint Button_Switch_SMD:SW_Push_1P1T_NO_6x6mm_H9.5mm -> Button_Switch_THT:SW_PUSH_6mm
Connections:
- net +5V_BATT: now also C19.2
- net FLASH_CS: now also R12.1; no longer U8.1 (~{CS})
- net USB_C_D_NEG: no longer D1.1 (L1), J1.A7 (D-), J1.B7 (D-)
- net USB_C_D_POS: no longer D1.3 (L2), J1.A6 (D+), J1.B6 (D+)
- net at C19.1, R5.2, R6.1: now also U7.5 (FB)
- new net: R12.2, U8.1 (~{CS})
- new net: D1.3 (L2), J1.A6 (D+), J1.B6 (D+)
- new net: D1.1 (L1), J1.A7 (D-), J1.B7 (D-)
Other:
- moved on the sheet: C15, C16, C17, C18, C19, C20, C21, C22, C23, C24, C25, D2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

Commit message: Add files via upload
Parts:
- removed SW1: SW_Push, Button_Switch_THT:SW_PUSH_6mm, symbol Switch:SW_Push
- added SW1: SW_SPDT, Button_Switch_SMD:SW_SPDT_PCM12, symbol Switch:SW_SPDT
- C1, C2, C28, C3, C33, C4, C5, C6, C7: LCSC PN (none) -> C1590
- C10, C11, C17: LCSC PN (none) -> C15849
- C12, C13: LCSC PN (none) -> C77020
- C14: LCSC PN (none) -> C1518208
- C15: LCSC PN (none) -> C2959727
- C16: LCSC PN (none) -> C64705
- C18, C32: LCSC PN (none) -> C5182432
- C19: LCSC PN (none) -> C107049
- C20, C21, C22, C23: LCSC PN (none) -> C2762594
- C24, C25: LCSC PN (none) -> C69335
- C26, C27: LCSC PN (none) -> C415535
- C29, C30: value 12pF -> 15pF; LCSC PN (none) -> C441742
- C31, C9: LCSC PN (none) -> C327204
- C34: LCSC PN (none) -> C107043
- C8: footprint Capacitor_SMD:C_0603_1608Metric -> Capacitor_SMD:C_0805_2012Metric; LCSC PN (none) -> C84416
- D1: LCSC PN (none) -> C15999
- D2: LCSC PN (none) -> C545548
- D3: LCSC PN (none) -> C2971978
- FB1: LCSC PN (none) -> C85824
- J1: footprint Connector_USB:USB_C_Receptacle_GCT_USB4105-xx-A_16P_TopMnt_Horizontal -> Connector_USB:USB_C_Receptacle_HCTL_HC-TYPE-C-16P-01A; LCSC PN (none) -> C2894897
- J2: LCSC PN (none) -> C98734
- J3, J4, J5, J6: LCSC PN (none) -> C306127
- J7: footprint Connector_PinSocket_2.54mm:PinSocket_1x06_P2.54mm_Vertical -> Connector_PinHeader_1.27mm:PinHeader_1x06_P1.27mm_Vertical; LCSC PN (none) -> C7470082
- L1: LCSC PN (none) -> C1329424
- R1, R2: LCSC PN (none) -> C125891
- R10: LCSC PN (none) -> C22809
- R11, R3: LCSC PN (none) -> C327797
- R12: footprint Resistor_SMD:R_0603_1608Metric -> Resistor_SMD:R_0402_1005Metric; LCSC PN (none) -> C327797
- R4, R5: LCSC PN (none) -> C14675
- R6: LCSC PN (none) -> C25962
- R7, R8: LCSC PN (none) -> C666957
- R9: LCSC PN (none) -> C21190
- SW2: footprint Button_Switch_THT:SW_PUSH_6mm -> Button_Switch_THT:SW_PUSH_6mm_H4.3mm; LCSC PN (none) -> C93157
- U1: LCSC PN (none) -> C15742
- U2: LCSC PN (none) -> C24112
- U3: footprint Package_LGA:Bosch_LGA-8_2x2.5mm_P0.65mm_ClockwisePinNumbering -> Custom Footprints:XDCR_BMP280; LCSC PN (none) -> C83291
- U4: LCSC PN (none) -> C150719
- U5: footprint Package_LGA:LGA-12_2x2mm_P0.5mm -> Custom Footprints:XDCR_LIS3MDL; LCSC PN (none) -> C478483
- U6: LCSC PN (none) -> C6332197
- U7: LCSC PN (none) -> C1852154
- U8: LCSC PN (none) -> C97521
- Y1: LCSC PN (none) -> C13738
Connections:
- net USB_C_D_NEG is gone; now on net USB_C_D_N: D1.6 (L1), U1.44 (PA11)
- net USB_C_D_POS is gone; now on net USB_C_D_P: D1.4 (L2), U1.45 (PA12)
- net +3.3V: now also SW1.1 (A)
- net BATT_SENSE: now also U1.9 (PC1); no longer U1.11 (PC3)
- net BOOT0: now also SW1.2 (B)
- net ESC_3: now also U1.56 (PB4); no longer U1.26 (PB0)
- net ESC_4: now also U1.57 (PB5); no longer U1.27 (PB1)
- net GND: now also SW1.3 (C)
- net IMU_INT: now also U1.33 (PB12); no longer U1.24 (PC4)
- net SCL: no longer U2.23 (SCL)
- net SDA: no longer U2.24 (SDA)
- net MPU_SDA: now reaches U1.40 (PC9)
- net MPU_SDA: now also U2.24 (SDA)
- net MPU_SCL: now reaches U1.41 (PA8)
- net MPU_SCL: now also U2.23 (SCL)
- net USB_C_D_P: now reaches D1.3 (L2), J1.A6 (D+), J1.B6 (D+)
- net USB_C_D_N: now reaches D1.1 (L1), J1.A7 (D-), J1.B7 (D-)
- no-connect marks 38 -> 36
Other:
- note removed: "Connectors/Switches"
- moved on the sheet: C1, C12, C13, C14, C15, C16, C17, C18, C19, C2, C20, C21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
