File: PCB/STM32F405_Flight_Controller.kicad_pcb (KiCad board)
At the start: 4 copper layers, 63.5 x 62.5 mm, 75 parts, among them J1 USB_C_Receptacle_USB2.0_16P, J2 XT60 (BATT), J3 ESC_1, J4 ESC_2, J5 ESC_3, J6 ESC_4, J7 SWD, J8 UART_External, SW1 SW_SPDT, SW2 SW_Push, U1 STM32F405RGTx, U4 AP7361C-33E, U5 LIS3MDL, U7 LMR33640DDDA, U8 W25Q128JVS, Y1 16MHz Crystal

Commit message: Add files via upload
Parts:
- removed C1, C2, C32: 100nF, Capacitor_SMD:C_0603_1608Metric
- removed C12, C13: 100nF, Capacitor_SMD:C_0402_1005Metric
- removed C14: 1uF, Capacitor_SMD:C_0402_1005Metric
- removed C31: 10nF, Capacitor_SMD:C_0603_1608Metric
- removed C33: 2.2u, Capacitor_SMD:C_0603_1608Metric
- removed J2: XT60 (BATT), Connector_AMASS:AMASS_XT60-F_1x02_P7.20mm_Vertical
- removed J3: ESC_1, Connector_PinSocket_2.54mm:PinSocket_1x03_P2.54mm_Vertical
- removed J4: ESC_2, Connector_PinSocket_2.54mm:PinSocket_1x03_P2.54mm_Vertical
- removed J5: ESC_3, Connector_PinSocket_2.54mm:PinSocket_1x03_P2.54mm_Vertical
- removed J6: ESC_4, Connector_PinSocket_2.54mm:PinSocket_1x03_P2.54mm_Vertical
- removed R12, R13, R14: 10k, Resistor_SMD:R_0603_1608Metric
- removed U2: ~, Custom Footprints:BMP390L
- removed U3: ~, Custom Footprints:XDCR_ICM-42670-P
- removed U5: LIS3MDL, Custom Footprints:XDCR_LIS3MDL
- removed U8: W25Q128JVS, Package_SO:SOIC-8_5.3x5.3mm_P1.27mm
- added C28: 100nF, Capacitor_SMD:C_0603_1608Metric, F.Cu at (290.7, 111.4)
- added C34: 100nF, Capacitor_SMD:C_0603_1608Metric, F.Cu at (210.9, 83.2)
- added C35: 100nF, Capacitor_SMD:C_0603_1608Metric, F.Cu at (208.5, 85.6)
- added C36: 1uF, Capacitor_SMD:C_0603_1608Metric, F.Cu at (242.2, 51.5)
- added C37: 10nF, Capacitor_SMD:C_0603_1608Metric, F.Cu at (222.6, 85.8)
- added C38: 100nF, Capacitor_SMD:C_0603_1608Metric, F.Cu at (242.2, 45.7)
- added C39: 0.1u, Capacitor_SMD:C_0603_1608Metric, F.Cu at (221.8, 82.5)
- added C40: 2.2u, Capacitor_SMD:C_0603_1608Metric, F.Cu at (223.5, 82.5)
- added C41: 100nF, Capacitor_SMD:C_0603_1608Metric, F.Cu at (242.1, 48.3)
- added J9: Conn_01x08, Connector_JST:JST_EH_B8B-EH-A_1x08_P2.50mm_Vertical, F.Cu at (211.4, 98.5)
- added R3: 10K, Resistor_SMD:R_0603_1608Metric, F.Cu at (294.7, 118.9)
- added SW1: SW_SPDT, Button_Switch_SMD:SW_SPDT_PCM12, F.Cu at (324.1, 132.1)
- added SW2: SW_Push, Button_Switch_THT:SW_PUSH_6mm_H4.3mm, F.Cu at (291.4, 124.7)
- added U11: ~, Custom Footprints:XDCR_ICM-42670-P, F.Cu at (219.5, 84.5)
- added U6: ~, Connector_PinHeader_2.54mm:PinHeader_1x04_P2.54mm_Vertical, F.Cu at (316.8, 131.4)
- added U9: ~, Custom Footprints:BMP390L, F.Cu at (211.1, 85.3)
- J8: value UART_External -> Conn_01x04; footprint Connector_JST:JST_EH_S4B-EH_1x04_P2.50mm_Horizontal -> Connector_JST:JST_EH_B4B-EH-A_1x04_P2.50mm_Vertical
- L1: footprint Inductor_SMD:L_Vishay_IHLP-4040 -> Inductor_SMD:L_Coilcraft_XAL7030-682
- moved R3 204.1 mm to (324.3, 152.4)
- moved SW1 204.1 mm to (324.3, 148.0)
- moved C28 204.1 mm to (323.9, 159.2)
- moved SW2 204.1 mm to (314.9, 156.6)
- moved D2 128.0 mm to (291.9, 142.0)
- moved R10 108.9 mm to (243.8, 57.5)
- moved R11 108.9 mm to (243.8, 55.7)
- moved U4 98.8 mm to (275.8, 93.5)
- moved C24 96.3 mm to (267.5, 92.5), turned to 0 degrees
- moved C25 95.9 mm to (267.5, 95.0), turned to 0 degrees
- moved D3 85.3 mm to (235.2, 47.9)
- moved R9 85.3 mm to (231.7, 47.9)
- moved J8 84.1 mm to (210.4, 58.3), turned to 0 degrees
- moved C6 82.1 mm to (227.2, 80.3), turned to 0 degrees
- moved H3 78.4 mm to (204.9, 93.6)
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Connections:
- R9 pad 1: Net-(D3-K) -> GND
- R9 pad 2: Net-(U1-PC5) -> Net-(D3-K)
- U1 pad 16: ESC_1 -> unconnected-(U1-PA2-Pad16)
- U1 pad 17: ESC_2 -> unconnected-(U1-PA3-Pad17)
- U1 pad 20: FLASH_CS -> unconnected-(U1-PA4-Pad20)
- U1 pad 21: SCK -> unconnected-(U1-PA5-Pad21)
- U1 pad 22: MISO -> unconnected-(U1-PA6-Pad22)
- U1 pad 23: MOSI -> unconnected-(U1-PA7-Pad23)
- U1 pad 25: Net-(U1-PC5) -> unconnected-(U1-PC5-Pad25)
- U1 pad 26: unconnected-(U1-PB0-Pad26) -> ESC_1
- U1 pad 27: unconnected-(U1-PB1-Pad27) -> ESC_2
- U1 pad 29: unconnected-(U1-PB10-Pad29) -> SCL
- U1 pad 30: unconnected-(U1-PB11-Pad30) -> SDA
- U1 pad 37: unconnected-(U1-PC6-Pad37) -> ESC_4
- U1 pad 38: unconnected-(U1-PC7-Pad38) -> ESC_3
- U1 pad 40: IMU_SDA -> unconnected-(U1-PC9-Pad40)
- U1 pad 41: IMU_SCL -> unconnected-(U1-PA8-Pad41)
- U1 pad 54: unconnected-(U1-PD2-Pad54) -> UART_ESC
- U1 pad 56: ESC_3 -> unconnected-(U1-PB4-Pad56)
- U1 pad 57: ESC_4 -> unconnected-(U1-PB5-Pad57)
- U1 pad 58: SCL -> unconnected-(U1-PB6-Pad58)
- U1 pad 59: SDA -> unconnected-(U1-PB7-Pad59)
Routing:
- net +3.3V: track 229.1 -> 18.5 mm, vias 24 -> 1
- net +5V: track 164.5 -> 0.00 mm, vias 6 -> 0
- net NRST: track 79.0 -> 12.3 mm, vias 4 -> 0
- net +BATT: track 56.4 -> 16.4 mm
- net GND: track 79.0 -> 45.6 mm, vias 60 -> 35
- net ESC_4: track 33.1 -> 0.00 mm, vias 2 -> 0
- net BMP_INT: track 27.8 -> 0.00 mm, vias 2 -> 0
- net Net-(U7-SW): track 25.7 -> 0.00 mm, vias 2 -> 0
- net ESC_3: track 23.3 -> 0.00 mm
- net Net-(D1-VP): track 20.5 -> 0.00 mm
- net Net-(U7-VCC): track 20.5 -> 0.00 mm, vias 2 -> 0
- net BATT_SENSE: track 20.3 -> 0.00 mm, vias 2 -> 0
- net BOOT0: track 22.6 -> 2.92 mm
- net ESC_1: track 19.3 -> 0.00 mm
- net MISO: track 19.2 -> 0.00 mm, vias 2 -> 0
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- removed copper zone on F.Cu, net +3.3V
- removed copper zone on F.Cu, net +5V
- removed copper zone on In1.Cu, net GND
Other:
- board outline removed
- board text removed: "SWD"
